Commit message: Prototype_2

File: Unity/Excavator/Assets/URDF/robot1.urdf (robot description, URDF)
Before this commit: robot onshape, 20 links, 19 joints
Links:
- link track_roller_wheel_1: mass 0 -> 5
- link track_roller_wheel_1_2: mass 0 -> 5
- link track_roller_wheel_1_3: mass 0 -> 5
- link track_roller_wheel_1_4: mass 0 -> 5
- link track_roller_wheel_1_5: mass 0 -> 5
- link track_roller_wheel_1_6: mass 0 -> 5

Commit message: code clean up

File: Unity/Excavator/Assets/URDF/robot1.urdf (robot description, URDF)
Before this commit: robot onshape, 20 links, 19 joints
Links:
- removed link carrier_roller
- removed link carrier_roller_2
- removed link track_roller_wheel_1
- removed link track_roller_wheel_1_2
- removed link track_roller_wheel_1_3
- removed link track_roller_wheel_1_4
- removed link track_roller_wheel_1_5
- removed link track_roller_wheel_1_6
Joints:
- removed joint idler1_wheel
- removed joint idler2_wheel
- removed joint roll_wheel_1
- removed joint roll_wheel_2
- removed joint roll_wheel_3
- removed joint roll_wheel_4
- removed joint roll_wheel_5
- removed joint roll_wheel_6
